File: AnalogSensorAmplifier/AnalogSensorAmplifier.kicad_sch (KiCad schematic)
At the start: 17 parts, among them J1 signal_in, J2 signal_out, U1 TLV9064

Commit message: Add BOM csv
Parts:
- RV1: value 1M -> PVG3A105C01R00
- U1: value TLV9064 -> TLV9154D
Changed lines of the file:
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@@
       (effects (font (size 1.27 1.27)) (justify left))
     )
-    (property "Value" "TLV9064" (at 38.1 46.99 0)
+    (property "Value" "TLV9154D" (at 38.1 46.99 0)
       (effects (font (size 1.27 1.27)) (justify left))
     )
@@
       (effects (font (size 1.27 1.27)) hide)
     )
-    (property "Datasheet" "https://www.ti.com/lit/ds/symlink/tlv9064.pdf" (at 40.64 40.64 0)
+    (property "Datasheet" "https://www.ti.com/lit/ds/symlink/tlv9154.pdf?ts=1711759780555" (at 40.64 40.64 0)
       (effects (font (size 1.27 1.27)) hide)
     )
@@
       (effects (font (size 1.27 1.27)))
     )
-    (property "Value" "TLV9064" (at 124.46 35.56 0)
+    (property "Value" "TLV9154D" (at 124.46 35.56 0)
       (effects (font (size 1.27 1.27)))
     )
@@
       (effects (font (size 1.27 1.27)) hide)
     )
-    (property "Datasheet" "https://www.ti.com/lit/ds/symlink/tlv9064.pdf" (at 125.73 33.02 0)
+    (property "Datasheet" "https://www.ti.com/lit/ds/symlink/tlv9154.pdf?ts=1711759780555" (at 125.73 33.02 0)
       (effects (font (size 1.27 1.27)) hide)
     )
@@
       (effects (font (size 1.27 1.27)))
     )
-    (property "Value" "TLV9064" (at 158.115 64.135 0)
+    (property "Value" "TLV9154D" (at 158.115 64.135 0)
       (effects (font (size 1.27 1.27)))
     )
@@
       (effects (font (size 1.27 1.27)) hide)
     )
-    (property "Datasheet" "https://www.ti.com/lit/ds/symlink/tlv9064.pdf" (at 159.385 62.23 0)
+    (property "Datasheet" "https://www.ti.com/lit/ds/symlink/tlv9154.pdf?ts=1711759780555" (at 159.385 62.23 0)
       (effects (font (size 1.27 1.27)) hide)
     )
@@
       (effects (font (size 1.27 1.27)))
     )
-    (property "Value" "TLV9064" (at 123.19 77.47 0)
+    (property "Value" "TLV9154D" (at 123.19 77.47 0)
       (effects (font (size 1.27 1.27)))
     )
@@
       (effects (font (size 1.27 1.27)) hide)
     )
-    (property "Datasheet" "https://www.ti.com/lit/ds/symlink/tlv9064.pdf" (at 124.46 74.93 0)
+    (property "Datasheet" "https://www.ti.com/lit/ds/symlink/tlv9154.pdf?ts=1711759780555" (at 124.46 74.93 0)
       (effects (font (size 1.27 1.27)) hide)
     )
@@
       (effects (font (size 1.27 1.27)))
     )
-    (property "Value" "TLV9064" (at 90.805 52.705 0)
+    (property "Value" "TLV9154D" (at 90.805 52.705 0)
       (effects (font (size 1.27 1.27)))
     )
@@
       (effects (font (size 1.27 1.27)) hide)
     )
-    (property "Datasheet" "https://www.ti.com/lit/ds/symlink/tlv9064.pdf" (at 92.075 50.165 0)
+    (property "Datasheet" "https://www.ti.com/lit/ds/symlink/tlv9154.pdf?ts=1711759780555" (at 92.075 50.165 0)
       (effects (font (size 1.27 1.27)) hide)
     )
@@
       (effects (font (size 1.27 1.27)) (justify right))
     )
-    (property "Value" "1M" (at 99.06 85.725 0)
-      (effects (font (size 1.27 1.27)) (justify right))
-    )
+    (property "Value" "PVG3A105C01R00" (at 99.06 85.725 0)
+      (effects (font (size 1.27 1.27)) (justify right))
+    )
